File: hardware/carrier-board/carrier.kicad_pcb (KiCad board)
At the start: 2 copper layers, 26 x 44 mm, 6 parts

Commit message: feat(hardware): v3 carrier board — route native USB D+/D- through J_PWR
Expands J_PWR to 4 pins (5V, GND, D+, D-), converting GP18/GP19 from
mechanical-only pads to real signal pads routed on-board. Lets the robot be
flashed and monitored over serial through the external Adafruit 5993 jack
(GND/D+/D-/5V per docs/hardware/interfaces.md's USB table) instead of
needing physical access to the ESP32-C3-Zero module's own onboard USB-C once
sealed inside the desk. Board stays 26x44mm. 0 DRC errors, 0 unconnected nets.

Co-Authored-By: Claude Sonnet 5 <noreply@anthropic.com>
Claude-Session: https://claude.ai/code/session_01NCfDjHNGeuiEoPta2KTLi3
Connections:
- J_ESP pad 15: (no net) -> USB_DM
- J_ESP pad 16: (no net) -> USB_DP
- J_PWR pad 2: 5V -> USB_DP
Routing:
- net USB_DP: track 0.00 -> 20.1 mm
- net USB_DM: track 0.00 -> 20.1 mm
- net 5V: track 75.0 -> 83.9 mm
