File: hardware/boards/compact-carrier-board/compact-carrier-board.kicad_pcb (KiCad board)
At the start: 2 copper layers, 26 x 44 mm, 7 parts

Commit message: fix(pcb): address CodeRabbit review — file naming, licensing, footprint metadata
- Rename board file to match its directory (compact-carrier-board.kicad_pcb),
  per the "directory name = project name" rule.
- Add hardware/boards/compact-carrier-board/** to REUSE.toml
  (CERN-OHL-S-2.0, Jon Truland) — was missing entirely on this branch.
- Fix docs/hardware/README.md -> docs/hardware/interfaces.md reference
  (the actual net-map file, not the overview).
- Re-origin all 7 footprints to their real pad-centroid (was (0,0) with
  absolute-coordinate pads), and set Value/LCSC on J_ESP1/J_ESP2 plus
  exclude_from_bom/exclude_from_pos_files on the 5 wire-only connectors.
  kicad-cli pcb export pos now reports (13.00, -1.65) / (13.00, -16.89)
  directly, matching the previously hand-derived values, with no manual
  patching needed.

Verified via kicad-cli (KiCad 10.0.5): DRC violations unchanged at 12/12
before and after (same set, only the origin-position readout differs) —
confirms the re-origin was a pure bookkeeping change with zero effect on
actual copper/silkscreen geometry.

Co-Authored-By: Claude Sonnet 5 <noreply@anthropic.com>
Claude-Session: https://claude.ai/code/session_01NCfDjHNGeuiEoPta2KTLi3
Parts:
- J_ESP1, J_ESP2: value (none) -> Kinghelm KH-2.54FH-1X9P-H3.5
- moved J_SERVO 40.6 mm to (16.8, 37.0)
- moved J_PWR 38.1 mm to (9.19, 37.0)
- moved J_I2C_PCA 31.0 mm to (7.92, 30.0)
- moved J_I2S 30.8 mm to (19.4, 24.0)
- moved J_I2C_OLED 25.3 mm to (7.92, 24.0)
- moved J_ESP2 21.3 mm to (13.0, 16.9)
- moved J_ESP1 13.1 mm to (13.0, 1.65)
